File: hardware/iot-cellular-risk-logger-stm32l4.kicad_sch (KiCad schematic)
At the start: 58 parts, among them J1 NanoSIM, J2 U.FL Antenna Connector (Male), J3 U.FL Antenna Connector (Male), J4 USB Type-C, J5 Conn_ARM_JTAG_SWD_10, Q1 IRLML6401, Q2 DTC143Z, U1 STM32L433CBUx, U2 SIM7070G, U3 W25Q64JV, U4 OPT3001DNPR, U5 SHT30-DIS, U6 MCP73831-2-OT, U7 L78L33ABUTR, U8 TXB0108PWR, U9 SMF05CT1G, Y1 SC-32S32.768

Commit message: schematics: add GSM, USART, level shifter, SIM nets&labels
Parts:
- removed C22: 100n, Capacitor_SMD:C_0603_1608Metric_Pad1.08x0.95mm_HandSolder, symbol Device:C
- removed J1: NanoSIM, personal:MOLEX_104224-0820, symbol 104224-0820:104224-0820
- removed U9: SMF05CT1G, Package_TO_SOT_SMD:SOT-363_SC-70-6, symbol SMF05CT1G:SMF05CT1G
- added C23: 100n, Capacitor_SMD:C_0603_1608Metric_Pad1.08x0.95mm_HandSolder, symbol Device:C
- added D4: SMF05CT1G, Package_TO_SOT_SMD:SOT-23-6, symbol Power_Protection:ESDA6V1-5SC6
- added J1: Nano SIM, personal:GCT_SIM8066-6-1-14-01-A_REVA, symbol SIM8066-6-1-14-01-A_REVA:SIM8066-6-1-14-01-A_REVA
- C6: value 1u -> 100n; footprint Capacitor_SMD:C_0805_2012Metric_Pad1.18x1.45mm_HandSolder -> Capacitor_SMD:C_0603_1608Metric_Pad1.08x0.95mm_HandSolder; LCSC Part C2932475 -> (none); Part CL21A105KACLNNC -> (none); URL https://www.lcsc.com/product-detail/Multilayer-Ceramic-Capa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 -> (none)
Connections:
- net VDDA is gone; now on net MCU_VDD: C5.1, C6.1, FB1.2
- net +3V3: no longer C7.1, C8.1, C9.1
- net GND: now also U1.23 (VSS), U1.35 (VSS), U1.47 (VSS), U1.49 (VSS), U1.8 (VSSA), U2.17 (GND), U2.18 (GND), U2.2 (GND), U2.29 (GND), U2.39 (GND), U2.45 (GND), U2.46 (GND), U2.54 (GND), U2.58 (GND), U2.59 (GND), U2.61 (GND), U2.62 (GND), U2.63 (GND), U2.64 (GND), U2.65 (GND), C23.1, D4.2 (GND), J1.C5 (GND), J1.G1 (GND), J1.G2 (GND), J1.G3 (GND), J1.G4 (GND)
- net PWRKEY: now also Q2.3 (C), U2.1 (PWRKEY); no longer Q2.1 (B)
- net SWDCLK: now also U1.37 (PA14)
- net SWDIO: now also U1.34 (PA13)
- net SWO: now also U1.39 (PB3)
- net _RESET: now also U1.7 (NRST)
- net LSE IN: now reaches C10.1, Y1.1
- net LSE IN: now also U1.3 (PC14)
- net LSE OUT: now reaches C11.1, Y1.2
- net LSE OUT: now also U1.4 (PC15)
- net RX: now reaches U8.1 (A1)
- net RX: now also U2.10 (UART1_RXD)
- net DTR3V: now reaches U8.12 (B7)
- net DTR3V: now also U1.28 (PB15)
- net RI3V: now reaches U8.13 (B6)
- net RI3V: now also U1.29 (PA8)
- net DCD3V: now reaches U8.14 (B5)
- net DCD3V: now also U1.27 (PB14)
- net CTS3V: now reaches U8.17 (B4)
- net CTS3V: now also U1.32 (PA11)
- net RTS3V: now reaches U8.18 (B3)
- net RTS3V: now also U1.33 (PA12)
- net RX3V: now reaches U8.19 (B2)
- net RX3V: now also U1.31 (PA10)
- net TX: now reaches U8.2 (A2)
- net TX: now also U2.9 (UART1_TXD)
- net TX3V: now reaches U8.20 (B1)
- net TX3V: now also U1.30 (PA9)
- net RTS: now reaches U8.3 (A3)
- net RTS: now also U2.8 (UART1_RTS)
- net CTS: now reaches U8.4 (A4)
- net CTS: now also U2.7 (UART1_CTS)
- net DCD: now reaches U8.7 (A5)
- net DCD: now also U2.5 (UART1_DCD)
- net RI: now reaches U8.8 (A6)
- net RI: now also U2.4 (UART1_RI)
- net DTR: now reaches U8.9 (A7)
- net DTR: now also U2.3 (UART1_DTR)
- net MCU_VDD: now reaches U1.24 (VDD)
- net MCU_VDD: now also C7.1, C8.1, C9.1, U1.36 (VDDUSB), U1.48 (VDD), U1.9 (VDDA)
- net VDD: now reaches U2.30 (SIM_VDD)
- net VDD: now also C23.2, D4.1 (IO1), J1.C1 (VCC)
- net DATA: now reaches U2.31 (SIM_DATA)
- net DATA: now also D4.5 (IO4), J1.C7 (I/O)
- net CLK: now reaches U2.32 (SIM_CLK)
- net CLK: now also D4.4 (IO3), J1.C3 (CLK)
- net RST: now reaches U2.33 (SIM_RST)
- net RST: now also D4.3 (IO2), J1.C2 (RST)
- net VBAT renamed GSM_VBAT
- new net GSM_PWR: Q2.1 (B)
- new net SIM_DETECT: J1.CD
- no-connect marks 3 -> 31
Other:
- note added: "CD disconects from GND on SIM insertion"
- note added: "TODO verify optimal TVS pins assignment"
- moved on the sheet: C10, C11, C12, C13, C14, C15, C16, C17, C21, C3, C7, C8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

Commit message: schematics: add QSPI, rework PMU, add sim, gsm, shifter nets
Parts:
- removed C18: 10u, Capacitor_SMD:C_0805_2012Metric_Pad1.18x1.45mm_HandSolder, symbol Device:C
- removed J3: U.FL Antenna Connector (Male), personal:HRS_U.FL-R-SMT_01_, symbol U.FL-R-SMT_01_:U.FL-R-SMT_01_
- removed NT1: NetTie_2, NetTie:NetTie-2_SMD_Pad0.5mm, symbol Device:NetTie_2
- removed R6: 47k, Resistor_SMD:R_0603_1608Metric_Pad0.98x0.95mm_HandSolder, symbol Device:R
- added AE1: GNSS Ceramic Antenna 25x25x4, personal:XDCR_APAE1590R2540AKDB1-T, symbol Device:Antenna
- added D5: BAT60A, Diode_SMD:D_SOD-323_HandSoldering, symbol Diode:BAT60A
- F1: value Polyfuse -> Polyfuse; footprint (none) -> Fuse:Fuse_1206_3216Metric_Pad1.42x1.75mm_HandSolder; LCSC Part # (none) -> C3157228; LCSC URL (none) -> https://www.lcsc.com/product-detail/Fuses_Littelfuse-046602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; Manufacturer (none) -> Littelfuse; Mfr. Part # (none) -> 046602.5NR
- J5: value Conn_ARM_JTAG_SWD_10 -> TagConnect SWD ARM
Connections:
- net +3V0: no longer C2.1, J5.1 (VTref), R4.1, U3.8 (VCC)
- net +3V3: now also C2.1, J5.1 (VTref), R4.1, U3.8 (VCC)
- net +5V: no longer C19.1, Q1.1 (G), R5.1, U7.3 (IN)
- net +BATT: now also C19.1, F1.2, U6.3 (V_{BAT}), U7.3 (IN); no longer Q1.2 (S)
- net BATTERY: no longer U6.3 (V_{BAT})
- net GND: now also J2.1 (GND), J2.2 (GND), R5.2
- net GPS_RF: now also AE1.1 (A)
- net QSPI_CLK: now also U1.13 (PA3)
- net QSPI_IO0: now also U1.19 (PB1)
- net QSPI_IO1: now also U1.18 (PB0)
- net QSPI_IO2: now also U1.17 (PA7)
- net QSPI_IO3: now also U1.16 (PA6)
- net USB_VBUS_SENSE: no longer R5.2
- net _QSPI_NCS: now also U1.12 (PA2)
- net at F1.1: now also Q1.2 (S)
- new net: Q1.1 (G), R5.1
Other:
- note added: "Q1 protects agains reverse polarity"
- note removed: "Q1 protects agains reverse polarity Q1 cuts off +BATT when USB 5V connected"
- note removed: "W25Q works down to 2V7, better to be 2V4"
- moved on the sheet: BT1, C10, C11, C2, C21, C3, C5, C6, C7, C8, C9, F1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

Commit message: PCB: manual RF routes done
Parts:
- removed C20: 10u, Capacitor_SMD:C_0805_2012Metric_Pad1.18x1.45mm_HandSolder, symbol Device:C
- removed D3: BZT52C4V7, Diode_SMD:D_SOD-123F, symbol Diode:BZT52Bxx
- removed D5: BAT60A, Diode_SMD:D_SOD-323_HandSoldering, symbol Diode:BAT60A
- removed F1: Polyfuse, Fuse:Fuse_1206_3216Metric_Pad1.42x1.75mm_HandSolder, symbol Device:Polyfuse
- removed FB2: 330, Resistor_SMD:R_0805_2012Metric_Pad1.20x1.40mm_HandSolder, symbol Device:FerriteBead_Small
- removed U2: SIM7070G, personal:MODULE_SIM7070G, symbol SIM7070G:SIM7070G
- removed U5: SHT30-DIS, Sensor_Humidity:Sensirion_DFN-8-1EP_2.5x2.5mm_P0.5mm_EP1.1x1.7mm, symbol Sensor_Humidity:SHT30-DIS
- removed U7: L78L33ABUTR, Package_TO_SOT_SMD:SOT-89-3, symbol Regulator_Linear:L78L33_SOT89
- added AE2: GSM Antenna, symbol Device:Antenna
- added BT2: Battery, Battery:BatteryHolder_Keystone_2462_2xAA, symbol Device:Battery
- added C18, C22, C24, C25, C26, C27: 100n, Capacitor_SMD:C_0603_1608Metric_Pad1.08x0.95mm_HandSolder, symbol Device:C
- added C28: 100p, Capacitor_SMD:C_0603_1608Metric_Pad1.08x0.95mm_HandSolder, symbol Device:C
- added C29, C30: 0p, Capacitor_SMD:C_0603_1608Metric, symbol Device:C
- added C31, C32: 10u, Capacitor_SMD:C_0805_2012Metric_Pad1.18x1.45mm_HandSolder, symbol Device:C
- added C33: 1n, Capacitor_SMD:C_0603_1608Metric_Pad1.08x0.95mm_HandSolder, symbol Device:C
- added D5: LED, LED_SMD:LED_0805_2012Metric_Pad1.15x1.40mm_HandSolder, symbol Device:LED
- added D6: TVS 5V, Diode_SMD:D_0603_1608Metric_Pad1.05x0.95mm_HandSolder, symbol Device:D_TVS
- added FB3: 330, Resistor_SMD:R_0805_2012Metric_Pad1.20x1.40mm_HandSolder, symbol Device:FerriteBead_Small
- added FL1: SAFFB1G56KB0F0A, Filter:Filter_1109-5_1.1x0.9mm, symbol Filter:SAFFB1G58KA0F0A
- added H1, H2, H3, H4: MountingHole_Pad, MountingHole:MountingHole_3.2mm_M3_Pad_Via, symbol Mechanical:MountingHole_Pad
- added JP1: SolderJumper_3_Bridged12, symbol Jumper:SolderJumper_3_Bridged12
- added L1: 8.2nH, Inductor_SMD:L_0603_1608Metric, symbol Device:L
- added L2, L3: 0L, Inductor_SMD:L_0603_1608Metric, symbol Device:L
- added L4: 1.5uH, Inductor_SMD:L_1008_2520Metric_Pad1.43x2.20mm_HandSolder, symbol Device:L
- added NT1, NT2, NT3, NT4, NT5, NT6, NT7: NetTie_2, NetTie:NetTie-2_SMD_Pad0.5mm, symbol Device:NetTie_2
- added R12, R6: 4k7, Resistor_SMD:R_0603_1608Metric_Pad0.98x0.95mm_HandSolder, symbol Device:R
- added R13, R14: 47k, Resistor_SMD:R_0603_1608Metric_Pad0.98x0.95mm_HandSolder, symbol Device:R
- added R15: 1k, Resistor_SMD:R_0805_2012Metric_Pad1.20x1.40mm_HandSolder, symbol Device:R
- added R16: 0R, Resistor_SMD:R_0603_1608Metric_Pad0.98x0.95mm_HandSolder, symbol Device:R
- added R17: 0R, Resistor_SMD:R_0603_1608Metric, symbol Device:R
- added R18: 1M, Resistor_SMD:R_0603_1608Metric_Pad0.98x0.95mm_HandSolder, symbol Device:R
- added U10: BGA 524N6 E6327, personal:BGA524N6E6327, symbol BGA_524N6_E6327:BGA_524N6_E6327
- added U11: BME280, Package_LGA:Bosch_LGA-8_2.5x2.5mm_P0.65mm_ClockwisePinNumbering, symbol Sensor:BME280
- added U2: LSM6DSO, personal:PQFN50P250X300X86-14N, symbol LSM6DSOX:LSM6DSOX
- added U5: TPS63051, personal:QFN50P250X250X100-12N, symbol TPS63051RMWR:TPS63051RMWR
- added U9: SIM7080G, personal:XCVR_SIM7080G, symbol SIM7080G:SIM7080G
- AE1: value GNSS Ceramic Antenna 25x25x4 -> GNSS Antenna; LCSC Part # C962216 -> C784398; LCSC URL https://www.lcsc.com/product-detail/Antennas_Shenzhen-Kingh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 -> https://www.lcsc.com/product-detail/Antennas_BAT-WIRELESS-B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; Manufacturer Shenzhen Kinghelm Elec -> BAT WIRELESS; Mfr. Part # KH-GPS252504-WY -> BWGNSCNX25-25W4
- BT1: value 18650 LiFePO4 -> 18650 Li-Ion; footprint Battery:BatteryHolder_Keystone_1042_1x18650 -> personal:BAT_BH-18650-PC; LCSC Part # C2988620 -> C19184083; LCSC URL https://www.lcsc.com/product-detail/Battery-Connectors_MYOUNG-BH-18650-B1BA002_C2988620.html -> https://www.lcsc.com/product-detail/Battery-Connectors_MYOUNG-BH-18650-A5BJ001-2D_C19184083.html; Mfr. Part # BH-18650-B1BA002 -> BH-18650-A5BJ001-2D
- FB1: LCSC Part C47130 -> (none); LCSC Part # (none) -> C47130; LCSC URL (none) -> https://www.lcsc.com/product-detail/Ferrite-Beads_Murata-El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; Manufacturer (none) -> Murata; Mfr. Part # (none) -> BLM21PG331SN1D; Part BLM21PG331SN1D -> (none); URL https://www.lcsc.com/product-detail/Ferrite-Beads_Murata-El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 -> (none)
- J2: value U.FL Antenna Connector (Male) -> U.FL; footprint personal:HRS_U.FL-R-SMT_01_ -> U.FL-R-SMT_01_:HRS_U.FL-R-SMT_01_; AVAILABILITY (none) -> Good; Availability (none) -> In Stock; Check_prices (none) -> https://www.snapeda.com/parts/U.FL-R-SMT(01)/Hirose+Electri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; DESCRIPTION (none) -> U.FL Series 6 Ghz 50 Ohm Ultra-small SMT Coaxial Cable Rece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; LCSC Part # C5137195 -> (none); LCSC URL https://www.lcsc.com/product-detail/RF-Connectors-Coaxial-C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 -> (none); MF (none) -> Hirose; MP (none) -> U.FL-R-SMT(01); Manufacturer BAT WIRELESS -> (none); Mfr. Part # BWU.FL-IPEX1 -> (none); PACKAGE (none) -> None; PRICE (none) -> 0.84 USD; Package (none) -> None; Price (none) -> None; Purchase-URL (none) -> https://www.snapeda.com/api/url_track_click_mouser/?unipart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; SnapEDA_Link (none) -> https://www.snapeda.com/parts/U.FL-R-SMT(01)/Hirose+Electri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
- R5: value 47k -> 100k
- R7: value 5k1 -> 2k5
- U4: footprint Personal:SON65P200X200X65-7N -> personal:SON65P200X200X65-7N; LCSC Part C90462 -> (none); LCSC Part # (none) -> C90462; LCSC URL (none) -> https://www.lcsc.com/product-detail/Ambient-Light-Sensors_T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; Mfr. Part # (none) -> OPT3001DNPR; Part OPT3001DNPR -> (none); URL https://www.lcsc.com/product-detail/Ambient-Light-Sensors_T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 -> (none)
- Y1: footprint Crystal:Crystal_SMD_EuroQuartz_EQ161-2Pin_3.2x1.5mm_HandSoldering -> Crystal:Crystal_SMD_EuroQuartz_EQ161-2Pin_3.2x1.5mm
Connections:
- net GSM_PWR is gone; now on net GSM_EN: Q2.1 (B)
- net +1V8: now also U9.40 (VDD_EXT)
- net +3V3: now also C4.1, C5.1, C6.1, C7.1, C8.1, C9.1, U1.24 (VDD), U1.36 (VDDUSB), U1.48 (VDD), U1.9 (VDDA), C18.1, C22.1, C24.1, C25.1, C26.1, C27.1, FB3.2, NT1.2, NT2.2, NT3.2, NT4.2, NT5.2, NT6.2, NT7.2, R12.1, R15.1, R18.1, R6.1; no longer FB1.1
- net +5V: now also R13.1
- net +BATT: now also FB1.2, Q1.2 (S), U5.10 (ILIM0), U5.11 (EN), U5.12 (VIN)
- net CHARGE_STAT: now also U1.40 (PB4)
- net CLK: now also U9.16 (SIM_CLK)
- net CTS: now also U9.4 (UART1_CTS)
- net CTS3V: now also U1.26 (PB13); no longer U1.32 (PA11)
- net DATA: now also U9.15 (SIM_DATA)
- net DCD: now also U8.3 (A3), U9.5 (UART1_DCD); no longer U8.7 (A5)
- net DCD3V: now also U1.29 (PA8), U8.18 (B3); no longer U1.27 (PB14), U8.14 (B5)
- net DTR: now also U8.2 (A2), U9.6 (UART1_DTR); no longer U8.9 (A7)
- net DTR3V: now also U8.19 (B2); no longer U8.12 (B7)
- net GND: now also BT2.2 (-), C18.2, C22.2, C24.2, C25.2, C26.2, C27.2, C29.2, C30.2, C31.2, C32.2, C33.2, D6.2 (A2), L2.2, L3.2, R14.2, U10.1 (GND_1), U10.4 (GND_2), U11.1 (GND), U11.5 (SDO), U11.7 (GND), U2.1 (SDO/SA0), U2.2 (SDX), U2.3 (SCX), U2.6 (GND), U2.7 (GND), U5.2 (GND), U5.6 (PFM/PWM), U5.9 (GND), U9.13 (GND), U9.19 (GND), U9.21 (GND), U9.27 (GND), U9.30 (GND), U9.31 (GND), U9.33 (GND), U9.36 (GND), U9.37 (GND), U9.45 (GND), U9.63 (GND), U9.66 (GND), U9.67 (GND), U9.69 (GND), U9.70 (GND), U9.71 (GND), U9.72 (GND), U9.73 (GND), U9.74 (GND), U9.75 (GND), U9.76 (GND), U9.77 (GND), U9.8 (GND)
- net GSM_RF: now also C29.1, R16.1, U9.32 (RF_ANT); no longer J2.3 (SIG)
- net RI: now also U8.1 (A1), U9.7 (UART1_RI); no longer U8.8 (A6)
- net RI3V: now also U1.27 (PB14), U8.20 (B1); no longer U1.29 (PA8), U8.13 (B6)
- net RST: now also U9.17 (SIM_RST)
- net RTS: now also U8.7 (A5), U9.3 (UART1_RTS); no longer U8.3 (A3)
- net RTS3V: now also U1.25 (PB12), U8.14 (B5); no longer U1.33 (PA12), U8.18 (B3)
- net RX: now also U8.8 (A6), U9.2 (UART1_RXD); no longer U8.1 (A1)
- net RX3V: now also U1.21 (PB10), U8.12 (B7); no longer U1.31 (PA10), U8.19 (B2)
- net SCL: now also U1.30 (PA9), R12.2, U11.4 (SCK), U2.13 (SCL)
- net SDA: now also U1.31 (PA10), R6.2, U11.3 (SDI), U2.14 (SDA)
- net SIM_DETECT: now also U1.20 (PB2)
- net TX: now also U8.9 (A7), U9.1 (UART1_TXD); no longer U8.2 (A2)
- net TX3V: now also U1.22 (PB11), U8.13 (B6); no longer U1.30 (PA9), U8.20 (B1)
- net USB_N: now also U1.32 (PA11)
- net USB_P: now also U1.33 (PA12)
- net VDD: now also U9.18 (SIM_VDD)
- net _LIGHT_INT: now also U1.41 (PB5)
- net USB_CC2: now reaches J4.B5 (CC2), R2.2
- net +VBUS: now reaches D1.2 (A), J4.A4 (VBUS), J4.A9 (VBUS), J4.B4 (VBUS), J4.B9 (VBUS)
- net USB_CC1: now reaches J4.A5 (CC1), R1.2
- net GND_SHIELD: now reaches C1.1, D2.1 (GND), J4.S1 (SHIELD), R3.1
- net GSM_EN: now reaches U1.10 (PA0)
- net GNSS_EN: now reaches U1.11 (PA1)
- net GNSS_EN: now also U10.6 (PON)
- net USB_VBUS: now reaches U1.38 (PA15)
- net USB_VBUS: now also R13.2, R14.1
- net IMU_INT1: now reaches U1.42 (PB6)
- net IMU_INT1: now also U2.4 (INT1)
- net IMU_INT2: now reaches U1.43 (PB7)
- net IMU_INT2: now also U2.9 (INT2)
- net +3V0: no longer names the net of U4.1 (VDD)
- net +3V0: now also NT4.1; no longer C4.1
- net BATTERY renamed +BATTERY
- net +BATTERY: now also BT2.1 (+)
- net GPS_RF renamed GNSS_ANT_RF
- net GNSS_ANT_RF: now also L2.1, R17.2
- net GSM_VBAT renamed +GSM_VBAT
- net +GSM_VBAT: now also FB1.1, U9.34 (VBAT), U9.35 (VBAT)
- removed net MCU_VDD: C5.1, C6.1, C7.1, C8.1, C9.1, FB1.2, U1.24 (VDD), U1.36 (VDDUSB), U1.48 (VDD), U1.9 (VDDA)
- net PWRKEY: no longer names the net of Q2.3 (C)
- net PWRKEY: now also U9.39 (PWRKEY)
- new net: C33.1, U5.7 (SS)
- new net: R18.2, U5.8 (PG)
- new net: NT3.1, U11.2 (CSB), U11.6 (VDDIO)
- new net: NT5.1, U2.12 (CS)
- new net: NT2.1, U2.5 (VDDIO)
- new net: NT1.1, U2.8 (VDD)
- new net: NT7.1, U11.8 (VDD)
- new net: FL1.2, FL1.5
- new net +LED: D5.2 (A), R15.2
- new net +VOUT: C31.1, C32.1, FB3.1, U5.4 (VOUT), U5.5 (FB)
- new net GNSS_M_RF: FL1.4, L3.1, R17.1
- new net GNSS_RF: U10.3 (AO), U9.68 (GNSS_ANT)
- new net GSM_ANT_RF: C28.2, D6.1 (A1), J2.3 (SIG)
- new net GSM_M_RF: C28.1, C30.1, R16.2
- new net IND1: L4.2, U5.1 (L1)
- new net IND2: L4.1, U5.3 (L2)
- new net LNA_RF: L1.1, U10.5 (AI)
- new net SAW_RF: FL1.1, L1.2
- new net VCC_LNA: NT6.1, U10.2 (VCC)
- new net _LED: D5.1 (K)
- no-connect marks 31 -> 47
Other:
- note added: "3D ACCELEROMETER & GYROSCOPE"
- note added: "4V2 BATTERY CHARGER"
- note added: "Alternative"
- note added: "BATTERY & MCU POWER"
- note added: "CD disconects from GND on SIM insertion SIM_DETECT becomes floating"
- note added: "Ceramic patch 25x25x4mm"
- note added: "Charge current: R7 PROG 2.5K: 400mA"
- note added: "I2C 0x6A, SA0(ADDR)=GND"
- note added: "I2C 0x76, SDO(ADDR)=GND"
- note added: "I2C 0x??, ADDR=GND"
- note added: "LNA"
- note added: "Nano SIM 1v8 card"
- note added: "RF Matching"
- note added: "SAW Filter"
- note added: "Standalone 6dbi LTE Antenna"
- note added: "TEMPERATURE & HUMIDITY & PRESSURE SENSOR"
- note added: "TODO make LED colour & current"
- note added: "TODO: boot pins connections"
- note added: "TODO: make a nice GND shield around the PCB"
- note added: "TODO; replace LED by RGB e.g. WS2812 ?"
- note added: "USB-C: DATA, CHARGE"
- note added: "level shifter 3v3 -> 1v8"
- note removed: "0x44, ADDR=L"
- note removed: "CD disconects from GND on SIM insertion"
- note removed: "Charge current: R7 PROG 5.1K: 200mA"
- note removed: "POWER MANAGEMENT"
- note removed: "SHT3x-DIS"
- note removed: "TEMPERATURE & HUMIDITY SENSOR"
- note removed: "VBAT NB-IoT: <0.6A VBAT EDGE/GPRS: <2A"
- moved on the sheet: BT1, C1, C10, C11, C12, C13, C14, C15, C16, C17, C19, C2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

Commit message: Schema: add boot0, reasign IMU INTs
Parts:
- removed JP1: SolderJumper_3_Bridged12, symbol Jumper:SolderJumper_3_Bridged12
- added J3: GSM_USB, Connector_PinHeader_2.54mm:PinHeader_1x04_P2.54mm_Vertical, symbol Connector:Conn_01x04_Pin
- added J6: GSM_DEBUG_UART, Connector_PinHeader_2.54mm:PinHeader_1x02_P2.54mm_Vertical, symbol Connector:Conn_01x02_Pin
- added JP1: SolderJumper_2_Open, Jumper:SolderJumper-2_P1.3mm_Open_RoundedPad1.0x1.5mm, symbol Jumper:SolderJumper_2_Open
- added R19: 10k, Resistor_SMD:R_0603_1608Metric_Pad0.98x0.95mm_HandSolder, symbol Device:R
- C10, C11: footprint Capacitor_SMD:C_0603_1608Metric_Pad1.08x0.95mm_HandSolder -> Capacitor_SMD:C_0603_1608Metric
- Y1: value SC-32S32.768 -> 32.768
Connections:
- net +3V3: now also JP1.1 (A)
- net GND: now also J3.1 (Pin_1), R19.1
- net IMU_INT1: now also U1.14 (PA4); no longer U1.42 (PB6)
- net IMU_INT2: now also U1.15 (PA5); no longer U1.43 (PB7)
- net _LED: now also U1.2 (PC13)
- net at U9.22 (UART2_TXD): now also J6.2 (Pin_2)
- net at U9.23 (UART2_RXD): now also J6.1 (Pin_1)
- net BOOT0: now reaches U1.44 (PH3)
- net BOOT0: now also JP1.2 (B), R19.2
- no-connect marks 47 -> 38
Other:
- note added: "Cload = 12p5 Cstray =~ 1p CX1 = CX2 = 2(12.5p - 1p) =~ 22p"
- note added: "TODO: add current measure break?"
- note added: "TODO: add debug i/o for current probe"
- note added: "TODO: add test point for I2C"
- note added: "short to loaf from USB"
- note removed: "TODO: boot pins connections"
- moved on the sheet: AE1, C26, C5, C6, C7, C8, C9, FL1, L1, L2, L3, R17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

Commit message: Schema: split to hierarchical schema
Parts:
- removed AE1: GNSS Antenna, personal:XDCR_APAE1590R2540AKDB1-T, symbol Device:Antenna
- removed AE2: GSM Antenna, symbol Device:Antenna
- removed BT1: 18650 Li-Ion, personal:BAT_BH-18650-PC, symbol Device:Battery_Cell
- removed BT2: Battery, Battery:BatteryHolder_Keystone_2462_2xAA, symbol Device:Battery
- removed C1: 4n7, Capacitor_SMD:C_0603_1608Metric_Pad1.08x0.95mm_HandSolder, symbol Device:C
- removed C10, C11: 22p, Capacitor_SMD:C_0603_1608Metric, symbol Device:C
- removed C12, C13, C18, C2, C21, C22, C23, C24, C25, C26, C27, C3, C4, C5, C6, C7, C8: 100n, Capacitor_SMD:C_0603_1608Metric_Pad1.08x0.95mm_HandSolder, symbol Device:C
- removed C14: 1u, Capacitor_SMD:C_0805_2012Metric_Pad1.18x1.45mm_HandSolder, symbol Device:C
- removed C15, C16, C17: 100uF, Capacitor_Tantalum_SMD:CP_EIA-3528-15_AVX-H_Pad1.50x2.35mm_HandSolder, symbol Device:C_Polarized
- removed C19, C31, C32, C9: 10u, Capacitor_SMD:C_0805_2012Metric_Pad1.18x1.45mm_HandSolder, symbol Device:C
- removed C28: 100p, Capacitor_SMD:C_0603_1608Metric_Pad1.08x0.95mm_HandSolder, symbol Device:C
- removed C29, C30: 0p, Capacitor_SMD:C_0603_1608Metric, symbol Device:C
- removed C33: 1n, Capacitor_SMD:C_0603_1608Metric_Pad1.08x0.95mm_HandSolder, symbol Device:C
- removed D1: BAT60A, Diode_SMD:D_SOD-323_HandSoldering, symbol Diode:BAT60A
- removed D2: PRTR5V0U2X, Package_TO_SOT_SMD:SOT-143, symbol Power_Protection:PRTR5V0U2X
- removed D4: SMF05CT1G, Package_TO_SOT_SMD:SOT-23-6, symbol Power_Protection:ESDA6V1-5SC6
- removed D5: LED, LED_SMD:LED_0805_2012Metric_Pad1.15x1.40mm_HandSolder, symbol Device:LED
- removed D6: TVS 5V, Diode_SMD:D_0603_1608Metric_Pad1.05x0.95mm_HandSolder, symbol Device:D_TVS
- removed FB1, FB3: 330, Resistor_SMD:R_0805_2012Metric_Pad1.20x1.40mm_HandSolder, symbol Device:FerriteBead_Small
- removed FL1: SAFFB1G56KB0F0A, Filter:Filter_1109-5_1.1x0.9mm, symbol Filter:SAFFB1G58KA0F0A
- removed J1: Nano SIM, personal:GCT_SIM8066-6-1-14-01-A_REVA, symbol SIM8066-6-1-14-01-A_REVA:SIM8066-6-1-14-01-A_REVA
- removed J2: U.FL, U.FL-R-SMT_01_:HRS_U.FL-R-SMT_01_, symbol U.FL-R-SMT_01_:U.FL-R-SMT_01_
- removed J3: GSM_USB, Connector_PinHeader_2.54mm:PinHeader_1x04_P2.54mm_Vertical, symbol Connector:Conn_01x04_Pin
- removed J4: USB Type-C, Connector_USB:USB_C_Receptacle_XKB_U262-16XN-4BVC11, symbol Connector:USB_C_Receptacle_USB2.0
- removed J5: TagConnect SWD ARM, Connector:Tag-Connect_TC2050-IDC-NL_2x05_P1.27mm_Vertical_with_bottom_clip, symbol Connector:Conn_ARM_JTAG_SWD_10
- removed J6: GSM_DEBUG_UART, Connector_PinHeader_2.54mm:PinHeader_1x02_P2.54mm_Vertical, symbol Connector:Conn_01x02_Pin
- removed JP1: SolderJumper_2_Open, Jumper:SolderJumper-2_P1.3mm_Open_RoundedPad1.0x1.5mm, symbol Jumper:SolderJumper_2_Open
- removed L1: 8.2nH, Inductor_SMD:L_0603_1608Metric, symbol Device:L
- removed L2, L3: 0L, Inductor_SMD:L_0603_1608Metric, symbol Device:L
- removed L4: 1.5uH, Inductor_SMD:L_1008_2520Metric_Pad1.43x2.20mm_HandSolder, symbol Device:L
- removed NT1, NT2, NT3, NT4, NT5, NT6, NT7: NetTie_2, NetTie:NetTie-2_SMD_Pad0.5mm, symbol Device:NetTie_2
- removed Q1: IRLML6401, Package_TO_SOT_SMD:SOT-23, symbol Device:Q_PMOS_GSD
- removed Q2: DTC143Z, Package_TO_SOT_SMD:SOT-23, symbol Transistor_BJT:DTC143Z
- removed R1, R2: 5k1, Resistor_SMD:R_0603_1608Metric_Pad0.98x0.95mm_HandSolder, symbol Device:R
- removed R10, R11, R13, R14, R8, R9: 47k, Resistor_SMD:R_0603_1608Metric_Pad0.98x0.95mm_HandSolder, symbol Device:R
- removed R12, R6: 4k7, Resistor_SMD:R_0603_1608Metric_Pad0.98x0.95mm_HandSolder, symbol Device:R
- removed R15: 1k, Resistor_SMD:R_0805_2012Metric_Pad1.20x1.40mm_HandSolder, symbol Device:R
- removed R16: 0R, Resistor_SMD:R_0603_1608Metric_Pad0.98x0.95mm_HandSolder, symbol Device:R
- removed R17: 0R, Resistor_SMD:R_0603_1608Metric, symbol Device:R
- removed R18, R3: 1M, Resistor_SMD:R_0603_1608Metric_Pad0.98x0.95mm_HandSolder, symbol Device:R
- removed R19, R4: 10k, Resistor_SMD:R_0603_1608Metric_Pad0.98x0.95mm_HandSolder, symbol Device:R
- removed R5: 100k, Resistor_SMD:R_0603_1608Metric_Pad0.98x0.95mm_HandSolder, symbol Device:R
- removed R7: 2k5, Resistor_SMD:R_0603_1608Metric_Pad0.98x0.95mm_HandSolder, symbol Device:R
- removed U1: STM32L433CBUx, Package_DFN_QFN:QFN-48-1EP_7x7mm_P0.5mm_EP5.6x5.6mm, symbol MCU_ST_STM32L4:STM32L433CBUx
- removed U10: BGA 524N6 E6327, personal:BGA524N6E6327, symbol BGA_524N6_E6327:BGA_524N6_E6327
- removed U11: BME280, Package_LGA:Bosch_LGA-8_2.5x2.5mm_P0.65mm_ClockwisePinNumbering, symbol Sensor:BME280
- removed U2: LSM6DSO, personal:PQFN50P250X300X86-14N, symbol LSM6DSOX:LSM6DSOX
- removed U3: W25Q64JV, Package_SO:SOIC-8_5.23x5.23mm_P1.27mm, symbol Memory_Flash:W25Q32JVSS
- removed U4: OPT3001DNPR, personal:SON65P200X200X65-7N, symbol OPT3001DNPR:OPT3001DNPR
- removed U5: TPS63051, personal:QFN50P250X250X100-12N, symbol TPS63051RMWR:TPS63051RMWR
- removed U6: MCP73831-2-OT, Package_TO_SOT_SMD:SOT-23-5, symbol Battery_Management:MCP73831-2-OT
- removed U8: TXB0108PWR, Package_SO:TSSOP-20_4.4x6.5mm_P0.65mm, symbol Logic_LevelTranslator:TXB0108DQSR
- removed U9: SIM7080G, personal:XCVR_SIM7080G, symbol SIM7080G:SIM7080G
- removed Y1: 32.768, Crystal:Crystal_SMD_EuroQuartz_EQ161-2Pin_3.2x1.5mm, symbol Device:Crystal
Connections:
- net GND: now also H1.1, H2.1, H3.1, H4.1
- no-connect marks 38 -> 0
Other:
- added sheet GSM Module (gsm.kicad_sch)
- added sheet MCU & Interfaces (mcu.kicad_sch)
- added sheet Power Management Unit (PMU) (pmu.kicad_sch)
- added sheet Sensors (sensors.kicad_sch)
- note removed: "3D ACCELEROMETER & GYROSCOPE"
- note removed: "4V2 BATTERY CHARGER"
- note removed: "AMBIENT LIGHT SENSOR"
- note removed: "Alternative"
- note removed: "BATTERY & MCU POWER"
- note removed: "BOM Field arr add to eeschema "Field Name Templates" according to https://www.pcbway.com/blog/PCB_Assembly/How_to_Build_a_BOM__Bill_Of_Materials_.html"
- note removed: "CD disconects from GND on SIM insertion SIM_DETECT becomes floating"
- note removed: "Ceramic patch 25x25x4mm"
- note removed: "Charge current: R7 PROG 2.5K: 400mA"
- note removed: "Cload = 12p5 Cstray =~ 1p CX1 = CX2 = 2(12.5p - 1p) =~ 22p"
- note removed: "D+/D- is differential pair Zdiff (differential impedance) is equal to 2 * Zodd, so a Zodd of 45 Ω gives us a Zdiff of 90 Ω"
- note removed: "I2C 0x6A, SA0(ADDR)=GND"
- note removed: "I2C 0x76, SDO(ADDR)=GND"
- note removed: "I2C 0x??, ADDR=GND"
- note removed: "LNA"
- note removed: "Nano SIM 1v8 card"
- note removed: "Preconditioning, Charge - L (0V) Charge complete - H (5V - 0V4)/2 = 2V3"
- note removed: "Q1 protects agains reverse polarity"
- note removed: "QSPI NOR FLASH 8MB"
- note removed: "RF Matching"
- note removed: "SAW Filter"
- note removed: "Standalone 6dbi LTE Antenna"
- note removed: "TEMPERATURE & HUMIDITY & PRESSURE SENSOR"
- note removed: "TODO make LED colour & current"
- note removed: "TODO verify optimal TVS pins assignment"
- note removed: "TODO: add current measure break?"
- note removed: "TODO: add debug i/o for current probe"
- note removed: "TODO: add test point for I2C"
- note removed: "TODO: check AN4879 Ann note about STM USB"
- note removed: "TODO: make a nice GND shield around the PCB"
- note removed: "TODO; replace LED by RGB e.g. WS2812 ?"
- note removed: "USB-C: DATA, CHARGE"
- note removed: "level shifter 3v3 -> 1v8"
- note removed: "short to loaf from USB"
- moved on the sheet: H1, H2, H3, H4
